File: $btshield.sch (KiCad schematic (older format))
At the start: 7 parts

Commit message: Arduino header added
Parts:
- added 3.3V: VCC, symbol VCC
- added GND: GND, symbol GND
- added P?: CONN_8, symbol CONN_8
- added R?: R, ~, symbol R
Connections:
- net labels removed: VCC
- wire segments 13 -> 15
Other:
- note added: "3.3V\n"
Changed lines of the file:
@@
 LIBS:valves
 LIBS:btshield
+LIBS:Arduino_As_Uno-cache
 EELAYER 27 0
 EELAYER END
@@
 Connection ~ 4950 4250
 $Comp
-L VCC #PWR?
+L VCC 3.3V
 U 1 1 55B1AB64
-P 6850 4300
-F 0 "#PWR?" H 6850 4400 30  0001 C CNN
-F 1 "VCC" H 6850 4400 30  0000 C CNN
-F 2 "" H 6850 4300 60  0000 C CNN
-F 3 "" H 6850 4300 60  0000 C CNN
-	1    6850 4300
+P 7000 4350
+F 0 "3.3V" H 7000 4450 30  0001 C CNN
+F 1 "VCC" H 7000 4450 30  0000 C CNN
+F 2 "" H 7000 4350 60  0000 C CNN
+F 3 "" H 7000 4350 60  0000 C CNN
+	1    7000 4350
 	1    0    0    -1
 $EndComp
@@
 	6550 5050 6550 5200
 Wire Wire Line
-	6850 4300 6850 4450
-Wire Wire Line
-	6850 4450 6550 4450
-Wire Wire Line
 	6400 4250 6550 4250
 Wire Wire Line
 	6550 4250 6550 4450
+$Comp
+L R R?
+U 1 1 55B1AC33
+P 6750 4150
+F 0 "R?" V 6830 4150 40  0000 C CNN
+F 1 "R" V 6757 4151 40  0000 C CNN
+F 2 "~" V 6680 4150 30  0000 C CNN
+F 3 "~" H 6750 4150 30  0000 C CNN
+	1    6750 4150
+	0    -1   -1   0
+$EndComp
+Wire Wire Line
+	7000 4350 6550 4350
+Connection ~ 6550 4350
+$Comp
+L GND GND
+U 1 1 55B1AC65
+P 7350 4250
+F 0 "GND" H 7350 4250 30  0001 C CNN
+F 1 "GND" H 7350 4180 30  0001 C CNN
+F 2 "" H 7350 4250 60  0000 C CNN
+F 3 "" H 7350 4250 60  0000 C CNN
+	1    7350 4250
+	1    0    0    -1
+$EndComp
+Wire Wire Line
+	7000 4150 7350 4150
+Wire Wire Line
+	7350 4150 7350 4250
+Wire Wire Line
+	6400 4150 6500 4150
+Text Notes 6850 4450 0    60   ~ 0
+3.3V\n
+$Comp
+L CONN_8 P?
+U 1 1 55B1B04B
+P 8450 3600
+F 0 "P?" V 8400 3600 60  0000 C CNN
+F 1 "CONN_8" V 8500 3600 60  0000 C CNN
+F 2 "" H 8450 3600 60  0000 C CNN
+F 3 "" H 8450 3600 60  0000 C CNN
+	1    8450 3600
+	1    0    0    1
+$EndComp
 $EndSCHEMATC
