File: $btshield.kicad_pcb (KiCad board)
At the start: 4 copper layers, 68.6 x 53.3 mm, 21 parts, among them Q1 BSS138, Q2 BSS138, SW1 SW_PUSH, SW2 SW_PUSH, SW3 SW_PUSH, SW4 SW_PUSH, SW5 SW_PUSH, U1 HC-10

Commit message: file dump 2, needs cleanup
Parts:
- renumbered SHIELD1 to BTSHIELD
Changed lines of the file:
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@@
     (links 56)
     (no_connects 1)
-    (area 148.514999 51.994999 217.245001 105.485001)
+    (area 143.84703 46.536 217.560501 105.86)
     (thickness 1.6)
     (drawings 5)
@@
     (2 UNUSED signal hide)
     (31 B.Cu signal)
+    (32 B.Adhes user)
     (33 F.Adhes user)
+    (34 B.Paste user)
     (35 F.Paste user)
+    (36 B.SilkS user)
     (37 F.SilkS user)
+    (38 B.Mask user)
     (39 F.Mask user)
     (40 Dwgs.User user)
@@
     (44 Edge.Cuts user)
     (45 Margin user)
+    (46 B.CrtYd user)
     (47 F.CrtYd user)
+    (48 B.Fab user)
     (49 F.Fab user)
   )
@@
     (visible_elements FFFFFF7F)
     (pcbplotparams
-      (layerselection 0x00020_80000001)
+      (layerselection 0x010f0_80000001)
       (usegerberextensions false)
       (excludeedgelayer true)
@@
       (net 4 /logic_converter/L_TX))
   )
-  (module btshield:arduino_shield locked (layer F.Cu)
+  (module btshield:arduino_shield (layer F.Cu)
     (at 148.59 105.41)
-    (fp_text reference SHIELD1 (at 2.54 -57.15) (layer F.SilkS)
+    (fp_text reference BTSHIELD (at 23.876 -3.048) (layer F.SilkS)
       (effects (font (thickness 0.3048)))
     )

Commit message: file dump 3
Routing:
- net +5V: track 145.3 -> 147.0 mm
- added copper zone on B.Cu, net GND
Changed lines of the file:
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@@
   (general
     (links 56)
-    (no_connects 1)
-    (area 143.84703 46.536 217.560501 105.86)
+    (no_connects 0)
+    (area 143.84703 49.076 218.694001 107.950001)
     (thickness 1.6)
     (drawings 5)
@@
       (effects (font (size 1 1) (thickness 0.15)))
     )
-    (fp_text value 1k (at 3.81 3.81 270) (layer F.Fab)
+    (fp_text value 1k (at 0 0 270) (layer F.Fab)
       (effects (font (size 1 1) (thickness 0.15)))
     )
@@
       (effects (font (size 1 1) (thickness 0.15)))
     )
-    (fp_text value 1k (at 3.81 3.81 270) (layer F.Fab)
+    (fp_text value 1k (at 0 0 270) (layer F.Fab)
       (effects (font (size 1 1) (thickness 0.15)))
     )
@@
       (effects (font (size 1 1) (thickness 0.15)))
     )
-    (fp_text value 1k (at 3.81 3.81 270) (layer F.Fab)
+    (fp_text value 1k (at 0.254 0 270) (layer F.Fab)
       (effects (font (size 1 1) (thickness 0.15)))
     )
@@
       (effects (font (size 1 1) (thickness 0.15)))
     )
-    (fp_text value 1k (at 3.81 3.81 270) (layer F.Fab)
+    (fp_text value 1k (at 0 0 270) (layer F.Fab)
       (effects (font (size 1 1) (thickness 0.15)))
     )
@@
       (effects (font (size 1 1) (thickness 0.15)))
     )
-    (fp_text value 1k (at 3.81 3.81 90) (layer F.Fab)
+    (fp_text value 1k (at 0 0 90) (layer F.Fab)
       (effects (font (size 1 1) (thickness 0.15)))
     )
@@
       (effects (font (size 1 1) (thickness 0.15)))
     )
-    (fp_text value 470 (at 3.81 3.81 180) (layer F.Fab)
+    (fp_text value 470 (at 0 0 180) (layer F.Fab)
       (effects (font (size 1 1) (thickness 0.15)))
     )
@@
       (effects (font (size 1 1) (thickness 0.15)))
     )
-    (fp_text value 10k (at 3.81 3.81 90) (layer F.Fab)
+    (fp_text value 10k (at 0.508 0 90) (layer F.Fab)
       (effects (font (size 1 1) (thickness 0.15)))
     )
@@
       (effects (font (size 1 1) (thickness 0.15)))
     )
-    (fp_text value 10k (at 3.81 3.81 90) (layer F.Fab)
+    (fp_text value 10k (at 0.508 0 90) (layer F.Fab)
       (effects (font (size 1 1) (thickness 0.15)))
     )
@@
     (descr "Resistor, Axial,  RM 10mm, 1/3W,")
     (tags "Resistor, Axial, RM 10mm, 1/3W,")
-    (fp_text reference R9 (at 0.24892 -3.50012) (layer F.SilkS)
-      (effects (font (size 1 1) (thickness 0.15)))
-    )
-    (fp_text value 10k (at 3.81 3.81) (layer F.Fab)
+    (fp_text reference R9 (at 0 -2.032) (layer F.SilkS)
+      (effects (font (size 1 1) (thickness 0.15)))
+    )
+    (fp_text value 10k (at 0 0) (layer F.Fab)
       (effects (font (size 1 1) (thickness 0.15)))
     )
@@
     (descr "Resistor, Axial,  RM 10mm, 1/3W,")
     (tags "Resistor, Axial, RM 10mm, 1/3W,")
-    (fp_text reference R10 (at 0.24892 -3.50012) (layer F.SilkS)
-      (effects (font (size 1 1) (thickness 0.15)))
-    )
-    (fp_text value 10k (at 3.81 3.81) (layer F.Fab)
+    (fp_text reference R10 (at 0 -2.032) (layer F.SilkS)
+      (effects (font (size 1 1) (thickness 0.15)))
+    )
+    (fp_text value 10k (at 0 0) (layer F.Fab)
       (effects (font (size 1 1) (thickness 0.15)))
     )
@@
   (gr_line (start 217.17 52.07) (end 217.17 105.41) (angle 90) (layer Edge.Cuts) (width 0.15))
   (gr_line (start 214.63 53.34) (end 213.36 52.07) (angle 90) (layer Edge.Cuts) (width 0.15))
-  (segment (start 197.104 98.044) (end 202.438 98.044) (width 0.25) (layer F.Cu) (net 1) (status 400000))
-  (segment (start 205.232 95.25) (end 205.232 92.71) (width 0.25) (layer F.Cu) (net 1) (status 800000))
+  (segment (start 197.104 98.044) (end 202.438 98.044) (width 0.25) (layer F.Cu) (net 1))
+  (segment (start 205.232 95.25) (end 205.232 92.71) (width 0.25) (layer F.Cu) (net 1))
   (segment (start 202.438 98.044) (end 205.232 95.25) (width 0.25) (layer F.Cu) (net 1))
   (segment (start 198.882 66.04) (end 205.994 66.04) (width 0.25) (layer B.Cu) (net 1))
@@
   (segment (start 205.994 72.09) (end 204.366 70.462) (width 0.25) (layer F.Cu) (net 4))
   (segment (start 204.366 70.462) (end 204.32 70.462) (width 0.25) (layer F.Cu) (net 4))
-  (segment (start 204.32 70.462) (end 204.216 70.358) (width 0.25) (layer F.Cu) (net 4))
-  (segment (start 204.216 70.358) (end 204.216 70.462) (width 0.25) (layer F.Cu) (net 4))
   (segment (start 209.28076 60.518) (end 209.616 60.518) (width 0.25) (layer F.Cu) (net 4))
   (segment (start 209.616 60.518) (end 211.328 62.23) (width 0.25) (layer F.Cu) (net 4))
@@
   (segment (start 192.81 68.858) (end 192.81 70.462) (width 0.25) (layer F.Cu) (net 6))
   (segment (start 189.484 65.532) (end 192.81 68.858) (width 0.25) (layer F.Cu) (net 6))
-  (segment (start 209.55 54.61) (end 209.55 56.134) (width 0.25) (layer B.Cu) (net 7) (status 400000))
-  (segment (start 198.13778 63.73622) (end 198.13778 61.722) (width 0.25) (layer F.Cu) (net 7) (status 800000))
+  (segment (start 209.55 54.61) (end 209.55 56.134) (width 0.25) (layer B.Cu) (net 7))
+  (segment (start 198.13778 63.73622) (end 198.13778 61.722) (width 0.25) (layer F.Cu) (net 7))
   (segment (start 197.866 64.008) (end 198.13778 63.73622) (width 0.25) (layer F.Cu) (net 7))
   (via (at 197.866 64.008) (size 0.6) (drill 0.4) (layers F.Cu B.Cu) (net 7))
@@
   (segment (start 189.738 88.392) (end 181.61 88.392) (width 0.25) (layer F.Cu) (net 13))
   (segment (start 193.04 91.694) (end 189.738 88.392) (width 0.25) (layer F.Cu) (net 13))
+  (segment (start 150.622 72.644) (end 151.13 72.644) (width 0.25) (layer F.Cu) (net 14))
+  (segment (start 151.13 72.644) (end 152.146 73.66) (width 0.25) (layer F.Cu) (net 14))
+  (segment (start 152.146 79.502) (end 150.622 81.026) (width 0.25) (layer F.Cu) (net 14))
+  (segment (start 152.146 73.66) (end 152.146 79.502) (width 0.25) (layer F.Cu) (net 14))
+  (segment (start 150.622 64.008) (end 151.892 65.278) (width 0.25) (layer F.Cu) (net 14))
+  (segment (start 152.146 71.12) (end 150.622 72.644) (width 0.25) (layer F.Cu) (net 14))
+  (segment (start 152.146 65.532) (end 152.146 71.12) (width 0.25) (layer F.Cu) (net 14))
+  (segment (start 151.892 65.278) (end 152.146 65.532) (width 0.25) (layer F.Cu) (net 14))
+  (segment (start 150.876 54.864) (end 151.13 54.864) (width 0.25) (layer F.Cu) (net 14))
+  (segment (start 151.13 54.864) (end 152.4 56.134) (width 0.25) (layer F.Cu) (net 14))
+  (segment (start 152.4 62.23) (end 150.622 64.008) (width 0.25) (layer F.Cu) (net 14))
+  (segment (start 152.4 56.134) (end 152.4 62.23) (width 0.25) (layer F.Cu) (net 14))
   (segment (start 150.876 54.864) (end 158.496 54.864) (width 0.25) (layer INTERNAL) (net 14))
   (segment (start 150.622 64.008) (end 158.242 64.008) (width 0.25) (layer INTERNAL) (net 14))
@@
   (segment (start 182.118 59.69) (end 182.118 64.262) (width 0.25) (layer B.Cu) (net 14))
   (segment (start 150.622 72.644) (end 150.622 73.152) (width 0.25) (layer F.Cu) (net 14))
-  (segment (start 150.622 73.152) (end 149.352 74.422) (width 0.25) (layer F.Cu) (net 14))
-  (segment (start 149.352 79.756) (end 150.622 81.026) (width 0.25) (layer F.Cu) (net 14))
-  (segment (start 149.352 74.422) (end 149.352 79.756) (width 0.25) (layer F.Cu) (net 14))
-  (segment (start 150.622 64.008) (end 149.352 65.278) (width 0.25) (layer F.Cu) (net 14))
-  (segment (start 150.622 71.882) (end 150.622 72.644) (width 0.25) (layer F.Cu) (net 14))
-  (segment (start 149.352 70.612) (end 150.622 71.882) (width 0.25) (layer F.Cu) (net 14))
-  (segment (start 149.352 65.278) (end 149.352 70.612) (width 0.25) (layer F.Cu) (net 14))
   (segment (start 150.876 54.864) (end 150.622 54.864) (width 0.25) (layer F.Cu) (net 14))
-  (segment (start 150.622 54.864) (end 149.352 56.134) (width 0.25) (layer F.Cu) (net 14))
-  (segment (start 149.352 56.134) (end 149.352 62.738) (width 0.25) (layer F.Cu) (net 14))
-  (segment (start 149.352 62.738) (end 150.622 64.008) (width 0.25) (layer F.Cu) (net 14))
+  (zone (net 2) (net_name GND) (layer B.Cu) (hatch edge 0.508)
+    (connect_pads (clearance 0.508))
+    (min_thickness 0.254)
+    (fill yes (arc_segments 16) (thermal_gap 0.508) (thermal_bridge_width 0.508))
+    (polygon
+      (pts
+        (xy 217.17 105.41) (xy 216.916 52.578) (xy 148.844 52.578) (xy 149.098 104.648) (xy 216.916 104.902)
+      )
+    )
+  )
 )
