File: btshield.kicad_pcb (KiCad board)
At the start: 4 copper layers, 68.6 x 53.3 mm, 21 parts, among them Q1 BSS138, Q2 BSS138, SW1 SW_PUSH, SW2 SW_PUSH, SW3 SW_PUSH, SW4 SW_PUSH, SW5 SW_PUSH, U1 HC-10

Commit message: fixed broken components (hopefully)
Parts:
- C1: value 0.1uF -> C
- turned R6 to 0 degrees
Connections:
- R6 pad 1: Net-(R6-Pad1) -> Net-(D1-Pad2)
- R6 pad 2: Net-(D1-Pad2) -> Net-(R6-Pad2)
- U1 pad 24: Net-(R6-Pad1) -> Net-(R6-Pad2)
Routing:
- net Net-(R6-Pad1): track 19.7 -> 0.00 mm
- net Net-(R6-Pad2): track 0.00 -> 19.7 mm
